Commit message: change mesh file URL

File: dynamixel_controller/urdf/d435.urdf.xacro (robot description, xacro)
@@ -7,5 +7,5 @@
 -->
 <robot name="sensor_d435" xmlns:xacro="http://ros.org/wiki/xacro">
-  <xacro:macro name="sensor_d435" params="parent *origin mesh_file">
+  <xacro:macro name="sensor_d435" params="parent *origin">
     <xacro:property name="M_PI" value="3.1415926535897931" />
     <!-- The following values are approximate, and the camera node
@@ -40,6 +40,5 @@
         <geometry>
           <!-- <box size="${d435_cam_width} ${d435_cam_height} ${d435_cam_depth}"/> -->
-	  <mesh filename="file://${mesh_file}" />
-          <!--<mesh filename="package://realsense2_camera/meshes/d435/d435.dae" />-->
+          <mesh filename="package://realsense2_camera/meshes/d435.dae" />
         </geometry>
         <material name="aluminum"/>

File: dynamixel_controller/urdf/pan_tilt.urdf.xacro (robot description, xacro)
@@ -2,5 +2,4 @@
 <robot name="pan_tilt_camera" xmlns:xacro="http://ros.org/wiki/xacro">
   <xacro:include filename="/urdf/d435.urdf.xacro"/>
-  <xacro:arg name="d435_mesh_file" default=""/>
   <link name="base_link">
     <visual>
@@ -16,6 +15,6 @@
     <visual>
       <geometry>
-        <!-- <cylinder length="0.6" radius="0.2"/> -->
-	<box size="0.04 0.03 0.05"/>
+        <mesh filename="package://dynamixel_urdf/meshes/ax12.stl" scale="0.001 0.001 0.001"/>
+	<!-- <box size="0.04 0.03 0.05"/> -->
       </geometry>
       <material name="green">
@@ -27,5 +26,6 @@
     <visual>
       <geometry>
-	<box size="0.04 0.03 0.05"/>
+        <mesh filename="package://dynamixel_urdf/meshes/ax12.stl" scale="0.001 0.001 0.001"/>
+	<!-- <box size="0.04 0.03 0.05"/> -->
       </geometry>
       <material name="red">
@@ -82,5 +82,5 @@
   </joint>
   -->
-  <sensor_d435 parent="camera_base_link" mesh_file="$(arg d435_mesh_file)">
+  <sensor_d435 parent="camera_base_link">
     <origin xyz="0.0 0.0 0.035" rpy="0 0 0"/>
   </sensor_d435>

Commit message: fix urdf

File: dynamixel_controller/urdf/d435.urdf.xacro (robot description, xacro)
@@ -40,5 +40,5 @@
         <geometry>
           <!-- <box size="${d435_cam_width} ${d435_cam_height} ${d435_cam_depth}"/> -->
-          <mesh filename="package://realsense2_camera/meshes/d435.dae" />
+          <mesh filename="file:/home/yokoyama/catkin_ws/src/realsense/realsense2_camera/meshes/d435.dae" />
         </geometry>
         <material name="aluminum"/>

File: dynamixel_controller/urdf/pan_tilt.urdf.xacro (robot description, xacro)
@@ -37,5 +37,5 @@
     <visual>
       <geometry>
-        <cylinder length="0.05" radius="0.02"/>
+        <!--<cylinder length="0.05" radius="0.02"/>-->
       </geometry>
       <material name="gray">
@@ -59,10 +59,10 @@
     <parent link="base_link"/>
     <child link="pan_link"/>
-    <origin xyz="0.01 0.0 0.04" rpy="0 -1.5708 0"/>
+    <origin xyz="0.0 0.0 0.04" rpy="1.5708 0 0"/>
   </joint>
   <joint name="pan_joint" type="revolute">
     <parent link="pan_link"/>
     <child link="tilt_link"/>
-    <origin xyz="0.05 0.0 0.01" rpy="0 1.5708 0"/>
+    <origin xyz="0.0 0.065 0.0" rpy="-1.5708 0 0"/>
     <axis xyz="0 0 1"/>
     <limit effort="1000.0" lower="-1.5" upper="1.5" velocity="0.5"/>
@@ -71,5 +71,5 @@
     <parent link="tilt_link"/>
     <child link="camera_base_link"/>
-    <origin xyz="0.0 0.0 0.02" rpy="0 0 -1.5708"/>
+    <origin xyz="0.0 0.0 0.0" rpy="0 0 0"/>
     <axis xyz="0 1 0"/>
     <limit effort="1000.0" lower="-1.5" upper="1.5" velocity="0.5"/>
@@ -83,5 +83,5 @@
   -->
   <sensor_d435 parent="camera_base_link">
-    <origin xyz="0.0 0.0 0.035" rpy="0 0 0"/>
+    <origin xyz="0.0 0.0 0.025" rpy="0 0 0"/>
   </sensor_d435>
 </robot>

Commit message: change mesh file path

File: dynamixel_controller/urdf/d435.urdf.xacro (robot description, xacro)
@@ -40,5 +40,5 @@
         <geometry>
           <!-- <box size="${d435_cam_width} ${d435_cam_height} ${d435_cam_depth}"/> -->
-          <mesh filename="file:/home/yokoyama/catkin_ws/src/realsense/realsense2_camera/meshes/d435.dae" />
+          <mesh filename="package://realsense2_camera/meshes/d435.dae" />
         </geometry>
         <material name="aluminum"/>
