Commit message: ros2 package

File: urdf/d435.urdf.xacro (robot description, xacro)
@@ -40,5 +40,5 @@
         <geometry>
           <!-- <box size="${d435_cam_width} ${d435_cam_height} ${d435_cam_depth}"/> -->
-          <mesh filename="package://realsense2_camera/meshes/d435.dae" />
+          <mesh filename="package://dynamixel_pantilt/meshes/d435.dae" />
         </geometry>
         <material name="aluminum"/>

File: urdf/pan_tilt.urdf.xacro (robot description, xacro)
@@ -1,5 +1,5 @@
 <?xml version="1.0"?>
 <robot name="pan_tilt_camera" xmlns:xacro="http://ros.org/wiki/xacro">
-  <xacro:include filename="/urdf/d435.urdf.xacro"/>
+  <xacro:include filename="package://dynamixel_pantilt/urdf/d435.urdf.xacro"/>
   <link name="base_link">
     <visual>
@@ -15,5 +15,5 @@
     <visual>
       <geometry>
-        <mesh filename="package://dynamixel_urdf/meshes/ax12.stl" scale="0.001 0.001 0.001"/>
+        <mesh filename="package://dynamixel_pantilt/meshes/ax12.stl" scale="0.001 0.001 0.001"/>
 	<!-- <box size="0.04 0.03 0.05"/> -->
       </geometry>

Commit message: fix errors

File: urdf/d435.urdf.xacro (robot description, xacro)
@@ -40,5 +40,5 @@
         <geometry>
           <!-- <box size="${d435_cam_width} ${d435_cam_height} ${d435_cam_depth}"/> -->
-          <mesh filename="package://dynamixel_pantilt/meshes/d435.dae" />
+          <mesh filename="../meshes/d435.dae" />
         </geometry>
         <material name="aluminum"/>

File: urdf/pan_tilt.urdf.xacro (robot description, xacro)
@@ -1,5 +1,6 @@
 <?xml version="1.0"?>
 <robot name="pan_tilt_camera" xmlns:xacro="http://ros.org/wiki/xacro">
-  <xacro:include filename="package://dynamixel_pantilt/urdf/d435.urdf.xacro"/>
+  <!--<xacro:include filename="package://dynamixel_pantilt/urdf/d435.urdf.xacro"/>-->
+  <xacro:include filename="d435.urdf.xacro"/>
   <link name="base_link">
     <visual>
@@ -15,5 +16,5 @@
     <visual>
       <geometry>
-        <mesh filename="package://dynamixel_pantilt/meshes/ax12.stl" scale="0.001 0.001 0.001"/>
+	<mesh filename="../meshes/ax12.stl" scale="0.001 0.001 0.001"/>
 	<!-- <box size="0.04 0.03 0.05"/> -->
       </geometry>
@@ -26,5 +27,5 @@
     <visual>
       <geometry>
-        <mesh filename="package://dynamixel_urdf/meshes/ax12.stl" scale="0.001 0.001 0.001"/>
+        <mesh filename="../meshes/ax12.stl" scale="0.001 0.001 0.001"/>
 	<!-- <box size="0.04 0.03 0.05"/> -->
       </geometry>

Commit message: fix errors

File: urdf/d435.urdf.xacro (robot description, xacro)
@@ -40,5 +40,5 @@
         <geometry>
           <!-- <box size="${d435_cam_width} ${d435_cam_height} ${d435_cam_depth}"/> -->
-          <mesh filename="../meshes/d435.dae" />
+	  <mesh filename="package://dynamixel_pantilt/meshes/d435.dae" />
         </geometry>
         <material name="aluminum"/>

File: urdf/pan_tilt.urdf.xacro (robot description, xacro)
@@ -16,5 +16,5 @@
     <visual>
       <geometry>
-	<mesh filename="../meshes/ax12.stl" scale="0.001 0.001 0.001"/>
+	<mesh filename="package://dynamixel_pantilt/meshes/ax12.stl" scale="0.001 0.001 0.001"/>
 	<!-- <box size="0.04 0.03 0.05"/> -->
       </geometry>
@@ -27,5 +27,5 @@
     <visual>
       <geometry>
-        <mesh filename="../meshes/ax12.stl" scale="0.001 0.001 0.001"/>
+	<mesh filename="package://dynamixel_pantilt/meshes/ax12.stl" scale="0.001 0.001 0.001"/>
 	<!-- <box size="0.04 0.03 0.05"/> -->
       </geometry>
